File: schematics/sauna-control.kicad_pcb (KiCad board)
At the start: 2 copper layers, 60 x 63 mm, 36 parts, among them U1 CPD-05231UR1_B, U2 LM1117-5.0, U3 ATmega88, X1 POWER, X2 SPI, X3 OUTPUT, X4 SENSORS

Commit message: Documentation improvements
Parts:
- B1: value Buzzer -> BUZZER
- R1, R2, R3, R4, R5, R6, R7, R8: value 150 -> 120
- R12, R13, R14, R16, R18, R19, R20: value 150 -> 200
- moved R11 67.2 mm to (112.7, 108.8)
- moved R14 67.2 mm to (105.9, 94.1)
- moved R15 67.2 mm to (105.9, 99.0)
- moved R16 67.2 mm to (112.7, 105.2)
- moved R18 67.2 mm to (127.0, 91.8)
- moved R19 67.2 mm to (127.0, 89.4)
- moved R3 67.2 mm to (104.9, 78.0)
- moved U2 67.2 mm to (130.2, 108.8)
- moved B1 67.2 mm to (143.8, 74.0)
- moved C1 67.2 mm to (121.9, 99.4)
- moved C2 67.2 mm to (110.9, 82.3)
- moved C3 67.2 mm to (122.0, 94.6)
- moved D1 67.2 mm to (96.1, 104.5)
- moved R1 67.2 mm to (119.5, 62.2)
- moved R10 67.2 mm to (119.8, 97.0)
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Connections:
- D1 pad 1: Net-(D1-Pad1) -> /ERROR_FIXING_JUMPER_WIRE
- R22 pad 2: Net-(D1-Pad1) -> /ERROR_FIXING_JUMPER_WIRE
- U3 pad 13: Net-(U3-Pad13) -> /ERROR_FIXING_JUMPER_WIRE
- U3 pad 19: Net-(D1-Pad1) -> /ERROR_FIXING_JUMPER_WIRE
- X4 pad 2: Net-(D1-Pad1) -> /ERROR_FIXING_JUMPER_WIRE
Routing:
- net /ERROR_FIXING_JUMPER_WIRE: track 0.00 -> 55.2 mm
- net Net-(D1-Pad1): track 55.2 -> 0.00 mm
Other:
- board text added: "1. +12V"
- board text added: "1. GND"
- board text added: "1. NC"
- board text added: "1. VCC"
- board text added: "2. CH2"
- board text added: "2. DATA"
- board text added: "2. GND"
- board text added: "2. VCC"
- board text added: "3. CH1"
- board text added: "3. GND"
- board text added: "3. MOSI"
- board text added: "4. GND"
- board text added: "4. MISO"
- board text added: "5. SCK"
- board text added: "6. RST"
