File: schematics/sauna-control.sch (KiCad schematic (older format))
At the start: 36 parts, among them U1 CPD-05231UR1_B, U2 LM1117-5.0, U3 ATmega88, X1 POWER, X2 SPI, X3 OUTPUT, X4 SENSORS

Commit message: Documentation improvements
Parts:
- R1, R2, R3, R4, R5, R6, R7, R8: value 150 -> 120
- R12, R13, R14, R16, R18, R19, R20: value 150 -> 200
Other:
- note added: "R1...R8\n 120"
Changed lines of the file:
@@
 encoding utf-8
 Sheet 1 1
-Title ""
-Date ""
-Rev ""
+Title "Sauna Control Module"
+Date "2020-05-23"
+Rev "A"
 Comp ""
 Comment1 ""
@@
 P 2400 2300
 F 0 "R1" H 1800 2450 50  0001 L CNN
-F 1 "150" H 1950 2450 50  0001 L CNN
+F 1 "120" H 1950 2450 50  0001 L CNN
 F 2 "Resistor_SMD:R_1206_3216Metric" V 2330 2300 50  0001 C CNN
 F 3 "~" H 2400 2300 50  0001 C CNN
@@
 P 2600 2300
 F 0 "R3" H 1950 2350 50  0001 L CNN
-F 1 "150" H 2100 2350 50  0001 L CNN
+F 1 "120" H 2100 2350 50  0001 L CNN
 F 2 "Resistor_SMD:R_1206_3216Metric" V 2530 2300 50  0001 C CNN
 F 3 "~" H 2600 2300 50  0001 C CNN
@@
 P 2800 2300
 F 0 "R5" H 2150 2350 50  0001 L CNN
-F 1 "150" H 2300 2350 50  0001 L CNN
+F 1 "120" H 2300 2350 50  0001 L CNN
 F 2 "Resistor_SMD:R_1206_3216Metric" V 2730 2300 50  0001 C CNN
 F 3 "~" H 2800 2300 50  0001 C CNN
@@
 P 3000 2300
 F 0 "R7" H 2350 2350 50  0001 L CNN
-F 1 "150" H 2500 2350 50  0001 L CNN
+F 1 "120" H 2500 2350 50  0001 L CNN
 F 2 "Resistor_SMD:R_1206_3216Metric" V 2930 2300 50  0001 C CNN
 F 3 "~" H 3000 2300 50  0001 C CNN
@@
 P 2500 1900
 F 0 "R2" H 1900 2050 50  0001 L CNN
-F 1 "150" H 2050 2050 50  0001 L CNN
+F 1 "120" H 2050 2050 50  0001 L CNN
 F 2 "Resistor_SMD:R_1206_3216Metric" V 2430 1900 50  0001 C CNN
 F 3 "~" H 2500 1900 50  0001 C CNN
@@
 P 2700 1900
 F 0 "R4" H 2050 1950 50  0001 L CNN
-F 1 "150" H 2200 1950 50  0001 L CNN
+F 1 "120" H 2200 1950 50  0001 L CNN
 F 2 "Resistor_SMD:R_1206_3216Metric" V 2630 1900 50  0001 C CNN
 F 3 "~" H 2700 1900 50  0001 C CNN
@@
 P 2900 1900
 F 0 "R6" H 2250 1950 50  0001 L CNN
-F 1 "150" H 2400 1950 50  0001 L CNN
+F 1 "120" H 2400 1950 50  0001 L CNN
 F 2 "Resistor_SMD:R_1206_3216Metric" V 2830 1900 50  0001 C CNN
 F 3 "~" H 2900 1900 50  0001 C CNN
@@
 P 3100 1900
 F 0 "R8" H 2450 1950 50  0001 L CNN
-F 1 "150" H 2600 1950 50  0001 L CNN
+F 1 "120" H 2600 1950 50  0001 L CNN
 F 2 "Resistor_SMD:R_1206_3216Metric" V 3030 1900 50  0001 C CNN
 F 3 "~" H 3100 1900 50  0001 C CNN
@@
 P 8550 1800
 F 0 "R19" V 8343 1800 50  0000 C CNN
-F 1 "150" V 8434 1800 50  0000 C CNN
+F 1 "200" V 8434 1800 50  0000 C CNN
 F 2 "Resistor_SMD:R_0603_1608Metric" V 8480 1800 50  0001 C CNN
 F 3 "~" H 8550 1800 50  0001 C CNN
@@
 P 8050 1900
 F 0 "R18" V 7750 1900 50  0000 C CNN
-F 1 "150" V 7850 1900 50  0000 C CNN
+F 1 "200" V 7850 1900 50  0000 C CNN
 F 2 "Resistor_SMD:R_0603_1608Metric" V 7980 1900 50  0001 C CNN
 F 3 "~" H 8050 1900 50  0001 C CNN
@@
 P 8550 2000
 F 0 "R20" V 8650 2000 50  0000 C CNN
-F 1 "150" V 8750 2000 50  0000 C CNN
+F 1 "200" V 8750 2000 50  0000 C CNN
 F 2 "Resistor_SMD:R_0603_1608Metric" V 8480 2000 50  0001 C CNN
 F 3 "~" H 8550 2000 50  0001 C CNN
@@
 P 6950 4250
 F 0 "R14" H 7100 4300 50  0000 C CNN
-F 1 "150" H 7100 4200 50  0000 C CNN
+F 1 "200" H 7100 4200 50  0000 C CNN
 F 2 "Resistor_SMD:R_1206_3216Metric" V 6880 4250 50  0001 C CNN
 F 3 "~" H 6950 4250 50  0001 C CNN
@@
 P 6750 4400
 F 0 "R12" H 6900 4350 50  0000 C CNN
-F 1 "150" H 6900 4450 50  0000 C CNN
+F 1 "200" H 6900 4450 50  0000 C CNN
 F 2 "Resistor_SMD:R_1206_3216Metric" V 6680 4400 50  0001 C CNN
 F 3 "~" H 6750 4400 50  0001 C CNN
@@
 P 7250 5100
 F 0 "R16" H 7400 5050 50  0000 C CNN
-F 1 "150" H 7400 5150 50  0000 C CNN
+F 1 "200" H 7400 5150 50  0000 C CNN
 F 2 "Resistor_SMD:R_1206_3216Metric" V 7180 5100 50  0001 C CNN
 F 3 "~" H 7250 5100 50  0001 C CNN
@@
 P 6800 1350
 F 0 "R13" V 7000 1350 50  0000 C CNN
-F 1 "150" V 6900 1350 50  0000 C CNN
+F 1 "200" V 6900 1350 50  0000 C CNN
 F 2 "Resistor_SMD:R_1206_3216Metric" V 6730 1350 50  0001 C CNN
 F 3 "~" H 6800 1350 50  0001 C CNN
@@
 Wire Wire Line
 	8650 6050 8650 3000
+Connection ~ 8650 3000
+Wire Wire Line
+	8650 3000 9000 3000
+Text Label 7000 6050 0    50   ~ 0
+ERROR_FIXING_JUMPER_WIRE
 Wire Bus Line
 	2700 4500 3900 4500
@@
 Wire Bus Line
 	2500 1350 3900 1350
-Connection ~ 8650 3000
-Wire Wire Line
-	8650 3000 9000 3000
-Text Label 7000 6050 0    50   ~ 0
-ERROR_FIXING_JUMPER_WIRE
+Text Notes 1950 2150 0    50   ~ 0
+R1...R8\n  120
 $EndSCHEMATC
